File: circuit/AutomaticPresentationTimer_v1.0/AutomaticPresentationTimer_v1.0.kicad_pcb (KiCad board)
At the start: 2 copper layers, 85.1 x 74.9 mm, 19 parts, among them J1 Conn_01x05, J2 Conn_01x03, J3 ZHO-0420S-05A4.5(5V), J4 ディスプレイモジュール, Q1 2SK4017, U1 Pico

Commit message: 2月4日作業分
Parts:
- moved J1 3.35 mm to (150.7, 103.6)
- moved J2 3.35 mm to (125.3, 106.1)
- moved TP6 2.11 mm to (145.2, 95.6)
Routing:
- net SW(GP12): track 42.8 -> 46.2 mm
- net +3.3V: track 157.8 -> 161.1 mm
- net B(GP11): track 36.7 -> 40.1 mm
- net A(GP10): track 42.1 -> 45.0 mm
- net GP15: track 33.7 -> 35.9 mm
Other:
- board text added: "B(GP11) GND A(GP10)"
- board text added: "GND 3.3V SCL SDA"
- board text added: "USB 給電"
- board text added: "× × SW(GP12) × 3.3V"
- board text removed: "VBUS"

Commit message: コンデンサの名称を修正
Parts:
- C1: value 1000µF 16V -> 1000µF 35V
Changed lines of the file:
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@@
 			)
 		)
-		(property "Value" "1000µF 16V"
+		(property "Value" "1000µF 35V"
 			(at 2.5 6.25 0)
 			(layer "F.Fab")
